File: ethernet_feather.kicad_pcb (KiCad board)
At the start: 0 parts

Commit message: Set basic PCB configuration
Parts:
- added A1: Adafruit_Feather_Generic, Module:Adafruit_Feather, F.Cu at (89.8, 74.7)
- added C1: 2pF, Capacitor_SMD:C_0603_1608Metric, F.Cu at (106.8, 126.2)
- added C10: 2.2µF, Capacitor_SMD:C_0603_1608Metric, F.Cu at (148.7, 83.8)
- added C11: 2.2nF, Capacitor_SMD:C_0603_1608Metric, F.Cu at (106.8, 123.7)
- added C12: 4.7µF, Capacitor_SMD:C_0603_1608Metric, F.Cu at (156.1, 75.3)
- added C13: 100nF, Capacitor_SMD:C_0603_1608Metric, F.Cu at (144.7, 86.3)
- added C14: 100nF, Capacitor_SMD:C_0603_1608Metric, F.Cu at (144.7, 83.8)
- added C15: 100nF, Capacitor_SMD:C_0603_1608Metric, F.Cu at (126.2, 106.1)
- added C16: 4.7µF, Capacitor_SMD:C_0603_1608Metric, F.Cu at (132.5, 104.1)
- added C17: 100nF, Capacitor_SMD:C_0603_1608Metric, F.Cu at (98.7, 125.8)
- added C18: 100nF, Capacitor_SMD:C_0603_1608Metric, F.Cu at (144.7, 88.8)
- added C19: 4.7µF, Capacitor_SMD:C_0603_1608Metric, F.Cu at (156.1, 77.8)
- added C2: 2pF, Capacitor_SMD:C_0603_1608Metric, F.Cu at (114.2, 113.0)
- added C20: 100nF, Capacitor_SMD:C_0603_1608Metric, F.Cu at (163.8, 68.8)
- added C21: 4.7µF, Capacitor_SMD:C_0603_1608Metric, F.Cu at (132.5, 101.6)
- added C22: 100nF, Capacitor_SMD:C_0603_1608Metric, F.Cu at (106.8, 121.2)
- added C23: 100nF, Capacitor_SMD:C_0603_1608Metric, F.Cu at (110.8, 123.7)
- added C24: 100nF, Capacitor_SMD:C_0603_1608Metric, F.Cu at (118.2, 113.0)
- added C3: 4pF, Capacitor_SMD:C_0603_1608Metric, F.Cu at (114.2, 110.5)
- added C4: 4pF, Capacitor_SMD:C_0603_1608Metric, F.Cu at (139.6, 95.1)
- added C5: C_Small, Capacitor_SMD:C_0603_1608Metric, F.Cu at (102.8, 125.7)
- added C6: 220nF, Capacitor_SMD:C_0603_1608Metric, F.Cu at (122.2, 110.5)
- added C7: 1µF, Capacitor_SMD:C_0603_1608Metric, F.Cu at (118.2, 115.5)
- added C8: 2.2µF, Capacitor_SMD:C_0603_1608Metric, F.Cu at (122.2, 108.0)
- added C9: 33nF, Capacitor_SMD:C_0603_1608Metric, F.Cu at (114.2, 118.0)
- added H1: 0.1", MountingHole:MountingHole_2.5mm_Pad, F.Cu at (134.3, 97.1)
- added H2: 0.1", MountingHole:MountingHole_2.5mm_Pad, F.Cu at (127.2, 101.6)
- added H3: 0.1", MountingHole:MountingHole_2.5mm, F.Cu at (150.8, 77.3)
- added H4: 0.1", MountingHole:MountingHole_2.5mm, F.Cu at (158.5, 70.8)
- added J1: USB_C_Receptacle_USB2.0, Connector_USB:USB_C_Receptacle_HRO_TYPE-C-31-M-12, F.Cu at (118.1, 97.0)
- added J2: TC2030-NL, Connector:Tag-Connect_TC2030-IDC-NL_2x03_P1.27mm_Vertical, F.Cu at (116.2, 104.2)
- added J3: Conn_01x02_MountingPin, Connector_JST:JST_PH_S2B-PH-SM4-TB_1x02-1MP_P2.00mm_Horizontal, F.Cu at (106.8, 77.5)
- added J4: RJ45_Abracon_ARJM11D7-114-AB-EW2, ethernet_feather:RJ45_Abracon_ARJM11D7-114, F.Cu at (122.3, 79.5)
- added J5: Conn_02x02_Odd_Even, Connector_PinSocket_2.54mm:PinSocket_2x02_P2.54mm_Vertical, F.Cu at (128.8, 93.5)
- added R1: 5.6kΩ, Resistor_SMD:R_0603_1608Metric, F.Cu at (118.2, 108.0)
- added R2: 5.6kΩ, Resistor_SMD:R_0603_1608Metric, F.Cu at (114.2, 115.5)
- added R3: 100kΩ, Resistor_SMD:R_0603_1608Metric, F.Cu at (110.8, 121.2)
- added R4: 120kΩ, Resistor_SMD:R_0603_1608Metric, F.Cu at (114.2, 108.0)
- added R5: 10kΩ, Resistor_SMD:R_0603_1608Metric, F.Cu at (118.2, 110.5)
- added TP1: D-2, TestPoint:TestPoint_Pad_D1.0mm, F.Cu at (121.8, 103.2)
- added TP2: D+2, TestPoint:TestPoint_Pad_D1.0mm, F.Cu at (121.8, 113.2)
- added U1: MIMXRT1051CVJ5B, ethernet_feather:LFBGA-196_12x12mm_Layout14x14_P0.8mm, F.Cu at (99.1, 92.1)
- added U2: LP3982IMM-3.3, Package_SO:VSSOP-8_3.0x3.0mm_P0.65mm, F.Cu at (95.6, 122.2)
- added U3: MCP73831-2-OT, Package_TO_SOT_SMD:SOT-23-5, F.Cu at (102.2, 122.2)
- added U4: W25Q32JVZP, Package_SON:WSON-8-1EP_6x5mm_P1.27mm_EP3.4x4.3mm, F.Cu at (96.2, 103.3)
- added U5: WE-TVS-82400102, Package_TO_SOT_SMD:SOT-23-6, F.Cu at (94.2, 126.8)
- added Y1: 24MHz 6pF, Crystal:Crystal_SMD_2016-4Pin_2.0x1.6mm, F.Cu at (126.2, 109.2)
- added Y2: 32.768kHz 7pF, Crystal:Crystal_SMD_MicroCrystal_MS3V-T1R, F.Cu at (89.6, 124.4)
Routing:
- net GND: track 0.00 -> 12.3 mm, vias 0 -> 15
- added copper zone on In1.Cu, net GND
Other:
- copper layers 0 -> 4
